Commit message: Version 1

File: 6DOF_URDF_description/urdf/6DOF_URDF.urdf (robot description, URDF)
Before this commit: robot 6DOF_URDF, 6 links, 5 joints
Links:
- removed link 20mm
- removed link Base_Motor
- removed link Elbow_Connector_Passive
- removed link Roll_Housing
- removed link UA_Motor
- added link Elbow, mass 0.733476; collision mesh filename=package://6DOF_URDF_description/meshes/6DOF_URDF/Elbow_coll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 scale=0.01 0.01 0.01; visual mesh filename=package://6DOF_URDF_description/meshes/6DOF_URDF/Elbow.dae scale=1 1 1
- added link Gripper, mass 0.011203; collision mesh filename=package://6DOF_URDF_description/meshes/6DOF_URDF/Gripper_co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 scale=0.01 0.01 0.01; visual mesh filename=package://6DOF_URDF_description/meshes/6DOF_URDF/Gripper.dae scale=1 1 1
- added link Roll, mass 0.682370; collision mesh filename=package://6DOF_URDF_description/meshes/6DOF_URDF/Roll_colli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 scale=0.01 0.01 0.01; visual mesh filename=package://6DOF_URDF_description/meshes/6DOF_URDF/Roll.dae scale=1 1 1
- added link Shoulder, mass 2.094136; collision mesh filename=package://6DOF_URDF_description/meshes/6DOF_URDF/Shoulder_c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 scale=0.01 0.01 0.01; visual mesh filename=package://6DOF_URDF_description/meshes/6DOF_URDF/Shoulder.d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 scale=1 1 1
- added link UA, mass 1.236306; collision mesh filename=package://6DOF_URDF_description/meshes/6DOF_URDF/UA_collisi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 scale=0.01 0.01 0.01; visual mesh filename=package://6DOF_URDF_description/meshes/6DOF_URDF/UA.dae scale=1 1 1
- added link Yaw, mass 0.259842; collision mesh filename=package://6DOF_URDF_description/meshes/6DOF_URDF/Yaw_collis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 scale=0.01 0.01 0.01; visual mesh filename=package://6DOF_URDF_description/meshes/6DOF_URDF/Yaw.dae scale=1 1 1
- link base_link: mass 0.601590 -> 0.596687
Joints:
- removed joint Rigid_25
- added joint Revolute_29: type revolute, parent UA, child Elbow, origin xyz=0.133252 0.154914 -0.036000 rpy=0.000000 0.000000 0.000000, axis 0.000000 0.000000 1.000000, limit lower=0.000000 upper=6.283185 effort=100.0 velocity=1.00
- added joint Revolute_46: type continuous, parent Yaw, child Gripper, origin xyz=-0.055454 -0.045134 0.050500 rpy=1.570796 0.110328 -0.887634, axis 0.000000 0.000000 1.000000, limit effort=100.0 velocity=1.00
- joint Revolute_13: child UA_Motor -> UA; origin xyz=0.076040 -0.153400 -0.055062 rpy=-1.570796 0.000000 0.000000 -> xyz=-0.007100 -0.149900 0.111900 rpy=1.570796 0.000000 0.086342; parent Base_Motor -> Shoulder
- joint Revolute_37: child Roll_Housing -> Roll; origin xyz=0.106612 0.079606 -0.186510 rpy=-1.570796 0.000000 -0.610865 -> xyz=-0.015463 0.083655 -0.071500 rpy=1.570796 -0.214197 -1.161568; parent Elbow_Connector_Passive -> Elbow
- joint Revolute_43: child 20mm -> Yaw; origin xyz=0.251183 -0.314427 0.170791 rpy=1.570796 -1.308997 0.000000 -> xyz=0.008683 0.049748 0.186000 rpy=1.570796 1.158599 -0.289463; parent Roll_Housing -> Roll
- joint Revolute_5: child Base_Motor -> Shoulder; origin xyz=-0.048850 0.117229 0.068000 rpy=0.000000 0.000000 0.000000 -> xyz=0.000000 0.000000 -0.051500 rpy=0.000000 0.000000 0.000000

File: 6DOF_URDF_description/urdf/6DOF_URDF.urdf.xacro (robot description, xacro)
@@ -5,7 +5,4 @@
     <color rgba="0.098 0.098 0.098 1.0"/>
   </material>
-  <material name="Steel">
-    <color rgba="1.000 1.000 1.000 1.0"/>
-  </material>
   <!-- Assembly includes -->
   <xacro:include filename="$(find 6DOF_URDF_description)/urdf/assemblies/6DOF_URDF.urdf.xacro"/>

File: 6DOF_URDF_description/urdf/assemblies/6DOF_URDF.urdf.xacro (robot description, xacro)
@@ -5,8 +5,8 @@
     <link name="${prefix}base_link">
       <inertial>
-        <origin xyz="-0.000000 0.000000 -0.031604" rpy="0 0 0"/>
-        <mass value="0.601590"/>
-        <inertia ixx="8.670932e-04" ixy="0.000000e+00" ixz="0.000000e+00"
-                 iyy="8.670932e-04" iyz="0.000000e+00" izz="1.232945e-03"/>
+        <origin xyz="0.000000 0.000000 -0.031884" rpy="0 0 0"/>
+        <mass value="0.596687"/>
+        <inertia ixx="8.608796e-04" ixy="0.000000e+00" ixz="0.000000e+00"
+                 iyy="8.608778e-04" iyz="0.000000e+00" izz="1.231935e-03"/>
       </inertial>
       <visual>
@@ -24,106 +24,121 @@
       </collision>
     </link>
-    <link name="${prefix}Base_Motor">
-      <inertial>
-        <origin xyz="0.049697 -0.108760 -0.020987" rpy="0 0 0"/>
-        <mass value="2.098842"/>
-        <inertia ixx="2.679976e-02" ixy="3.861349e-03" ixz="-5.600426e-04"
-                 iyy="3.790863e-03" iyz="1.696564e-03" izz="2.827367e-02"/>
-      </inertial>
-      <visual>
-        <origin xyz="0.000000 0.000000 -0.000600" rpy="3.141593 0.000000 0.000000"/>
-        <geometry>
-          <mesh filename="package://6DOF_URDF_description/meshes/6DOF_URDF/Base_Motor.dae" scale="1 1 1"/>
-        </geometry>
-        <material name="Steel"/>
-      </visual>
-      <collision>
-        <origin xyz="0.000000 0.000000 -0.000600" rpy="3.141593 0.000000 0.000000"/>
-        <geometry>
-          <mesh filename="package://6DOF_URDF_description/meshes/6DOF_URDF/Base_Motor_collision.stl" scale="0.01 0.01 0.01"/>
-        </geometry>
-      </collision>
-    </link>
-    <link name="${prefix}UA_Motor">
-      <inertial>
-        <origin xyz="-0.081949 -0.130878 0.071799" rpy="0 0 0"/>
-        <mass value="1.315683"/>
-        <inertia ixx="5.586235e-03" ixy="-2.437625e-03" ixz="1.020418e-04"
-                 iyy="4.787916e-03" iyz="1.483998e-04" izz="5.396456e-03"/>
-      </inertial>
-      <visual>
-        <origin xyz="-0.077066 -0.122959 0.060400" rpy="-3.141593 0.000000 2.443461"/>
-        <geometry>
-          <mesh filename="package://6DOF_URDF_description/meshes/6DOF_URDF/UA_Motor.dae" scale="1 1 1"/>
-        </geometry>
-        <material name="Steel"/>
-      </visual>
-      <collision>
-        <origin xyz="-0.077066 -0.122959 0.060400" rpy="-3.141593 0.000000 2.443461"/>
-        <geometry>
-          <mesh filename="package://6DOF_URDF_description/meshes/6DOF_URDF/UA_Motor_collision.stl" scale="0.01 0.01 0.01"/>
-        </geometry>
-      </collision>
-    </link>
-    <link name="${prefix}Elbow_Connector_Passive">
-      <inertial>
-        <origin xyz="-0.019245 0.011518 0.062617" rpy="0 0 0"/>
-        <mass value="3.223631"/>
-        <inertia ixx="4.864071e-03" ixy="3.444810e-03" ixz="3.038557e-04"
-                 iyy="8.503665e-03" iyz="-1.358472e-04" izz="9.997296e-03"/>
-      </inertial>
-      <visual>
-        <origin xyz="0.000000 0.000000 0.000000" rpy="0.000000 0.000000 0.000000"/>
-        <geometry>
-          <mesh filename="package://6DOF_URDF_description/meshes/6DOF_URDF/Elbow_Connector_Passive.dae" scale="1 1 1"/>
-        </geometry>
-        <material name="Steel"/>
-      </visual>
-      <collision>
-        <origin xyz="0.000000 0.000000 0.000000" rpy="0.000000 0.000000 0.000000"/>
-        <geometry>
-          <mesh filename="package://6DOF_URDF_description/meshes/6DOF_URDF/Elbow_Connector_Passive_collision.stl" scale="0.01 0.01 0.01"/>
-        </geometry>
-      </collision>
-    </link>
-    <link name="${prefix}Roll_Housing">
-      <inertial>
-        <origin xyz="0.041154 -0.253297 -0.010541" rpy="0 0 0"/>
-        <mass value="0.777648"/>
-        <inertia ixx="2.292696e-03" ixy="1.323394e-06" ixz="-2.147043e-06"
-                 iyy="1.753582e-03" iyz="-2.028961e-04" izz="8.080313e-04"/>
-      </inertial>
-      <visual>
-        <origin xyz="0.041229 -0.283510 -0.047460" rpy="-1.570796 1.570796 0.000000"/>
-        <geometry>
-          <mesh filename="package://6DOF_URDF_description/meshes/6DOF_URDF/Roll_Housing.dae" scale="1 1 1"/>
-        </geometry>
-        <material name="Steel"/>
-      </visual>
-      <collision>
-        <origin xyz="0.041229 -0.283510 -0.047460" rpy="-1.570796 1.570796 0.000000"/>
-        <geometry>
-          <mesh filename="package://6DOF_URDF_description/meshes/6DOF_URDF/Roll_Housing_collision.stl" scale="0.01 0.01 0.01"/>
-        </geometry>
-      </collision>
-    </link>
-    <link name="${prefix}20mm">
-      <inertial>
-        <origin xyz="-0.160624 0.152440 -0.069417" rpy="0 0 0"/>
-        <mass value="0.318715"/>
-        <inertia ixx="1.638087e-04" ixy="5.662339e-05" ixz="-3.202578e-11"
-                 iyy="1.870873e-04" iyz="-1.709404e-10" izz="2.324443e-04"/>
-      </inertial>
-      <visual>
-        <origin xyz="-0.184366 0.172623 -0.069417" rpy="2.443461 -1.570796 0.000000"/>
-        <geometry>
-          <mesh filename="package://6DOF_URDF_description/meshes/6DOF_URDF/20mm.dae" scale="1 1 1"/>
-        </geometry>
-        <material name="Steel"/>
-      </visual>
-      <collision>
-        <origin xyz="-0.184366 0.172623 -0.069417" rpy="2.443461 -1.570796 0.000000"/>
-        <geometry>
-          <mesh filename="package://6DOF_URDF_description/meshes/6DOF_URDF/20mm_collision.stl" scale="0.01 0.01 0.01"/>
+    <link name="${prefix}Shoulder">
+      <inertial>
+        <origin xyz="-0.000095 -0.008184 0.098482" rpy="0 0 0"/>
+        <mass value="2.094136"/>
+        <inertia ixx="2.587229e-02" ixy="5.786696e-03" ixz="7.038970e-04"
+                 iyy="4.623819e-03" iyz="-1.651409e-03" izz="2.818176e-02"/>
+      </inertial>
+      <visual>
+        <origin xyz="0.000000 0.000000 0.000000" rpy="0.000000 0.000000 0.086342"/>
+        <geometry>
+          <mesh filename="package://6DOF_URDF_description/meshes/6DOF_URDF/Shoulder.dae" scale="1 1 1"/>
+        </geometry>
+      </visual>
+      <collision>
+        <origin xyz="0.000000 0.000000 0.000000" rpy="0.000000 0.000000 0.086342"/>
+        <geometry>
+          <mesh filename="package://6DOF_URDF_description/meshes/6DOF_URDF/Shoulder_collision.stl" scale="0.01 0.01 0.01"/>
+        </geometry>
+      </collision>
+    </link>
+    <link name="${prefix}UA">
+      <inertial>
+        <origin xyz="0.070469 0.078205 -0.113480" rpy="0 0 0"/>
+        <mass value="1.236306"/>
+        <inertia ixx="4.958228e-03" ixy="-2.087939e-03" ixz="-1.318650e-07"
+                 iyy="4.306581e-03" iyz="-2.819097e-05" izz="4.648503e-03"/>
+      </inertial>
+      <visual>
+        <origin xyz="0.000000 0.000000 0.000000" rpy="0.000000 0.000000 -0.698132"/>
+        <geometry>
+          <mesh filename="package://6DOF_URDF_description/meshes/6DOF_URDF/UA.dae" scale="1 1 1"/>
+        </geometry>
+      </visual>
+      <collision>
+        <origin xyz="0.000000 0.000000 0.000000" rpy="0.000000 0.000000 -0.698132"/>
+        <geometry>
+          <mesh filename="package://6DOF_URDF_description/meshes/6DOF_URDF/UA_collision.stl" scale="0.01 0.01 0.01"/>
+        </geometry>
+      </collision>
+    </link>
+    <link name="${prefix}Elbow">
+      <inertial>
+        <origin xyz="-0.015531 0.020790 -0.069395" rpy="0 0 0"/>
+        <mass value="0.733476"/>
+        <inertia ixx="1.328959e-03" ixy="4.778990e-04" ixz="-2.397529e-05"
+                 iyy="7.168999e-04" iyz="3.209492e-05" izz="1.533380e-03"/>
+      </inertial>
+      <visual>
+        <origin xyz="0.000000 0.000000 0.000000" rpy="0.000000 0.000000 -0.698132"/>
+        <geometry>
+          <mesh filename="package://6DOF_URDF_description/meshes/6DOF_URDF/Elbow.dae" scale="1 1 1"/>
+        </geometry>
+      </visual>
+      <collision>
+        <origin xyz="0.000000 0.000000 0.000000" rpy="0.000000 0.000000 -0.698132"/>
+        <geometry>
+          <mesh filename="package://6DOF_URDF_description/meshes/6DOF_URDF/Elbow_collision.stl" scale="0.01 0.01 0.01"/>
+        </geometry>
+      </collision>
+    </link>
+    <link name="${prefix}Roll">
+      <inertial>
+        <origin xyz="-0.001708 -0.009290 0.127780" rpy="0 0 0"/>
+        <mass value="0.682370"/>
+        <inertia ixx="1.825964e-03" ixy="-6.698787e-05" ixz="-2.868309e-05"
+                 iyy="1.445666e-03" iyz="-1.542829e-04" izz="6.361788e-04"/>
+      </inertial>
+      <visual>
+        <origin xyz="0.000000 0.000000 0.000000" rpy="3.141593 0.000000 -0.214197"/>
+        <geometry>
+          <mesh filename="package://6DOF_URDF_description/meshes/6DOF_URDF/Roll.dae" scale="1 1 1"/>
+        </geometry>
+      </visual>
+      <collision>
+        <origin xyz="0.000000 0.000000 0.000000" rpy="3.141593 0.000000 -0.214197"/>
+        <geometry>
+          <mesh filename="package://6DOF_URDF_description/meshes/6DOF_URDF/Roll_collision.stl" scale="0.01 0.01 0.01"/>
+        </geometry>
+      </collision>
+    </link>
+    <link name="${prefix}Yaw">
+      <inertial>
+        <origin xyz="-0.015546 -0.012336 0.050500" rpy="0 0 0"/>
+        <mass value="0.259842"/>
+        <inertia ixx="1.293116e-04" ixy="-3.743600e-05" ixz="-3.755642e-12"
+                 iyy="1.422665e-04" iyz="1.808699e-10" izz="1.729664e-04"/>
+      </inertial>
+      <visual>
+        <origin xyz="0.000000 0.000000 0.000000" rpy="-3.141593 0.000000 -0.412197"/>
+        <geometry>
+          <mesh filename="package://6DOF_URDF_description/meshes/6DOF_URDF/Yaw.dae" scale="1 1 1"/>
+        </geometry>
+      </visual>
+      <collision>
+        <origin xyz="0.000000 0.000000 0.000000" rpy="-3.141593 0.000000 -0.412197"/>
+        <geometry>
+          <mesh filename="package://6DOF_URDF_description/meshes/6DOF_URDF/Yaw_collision.stl" scale="0.01 0.01 0.01"/>
+        </geometry>
+      </collision>
+    </link>
+    <link name="${prefix}Gripper">
+      <inertial>
+        <origin xyz="0.000000 0.000000 -0.014692" rpy="0 0 0"/>
+        <mass value="0.011203"/>
+        <inertia ixx="1.935595e-06" ixy="0.000000e+00" ixz="0.000000e+00"
+                 iyy="1.935595e-06" iyz="0.000000e+00" izz="1.864791e-06"/>
+      </inertial>
+      <visual>
+        <origin xyz="0.000000 0.000000 0.000000" rpy="0.000000 0.000000 -0.607892"/>
+        <geometry>
+          <mesh filename="package://6DOF_URDF_description/meshes/6DOF_URDF/Gripper.dae" scale="1 1 1"/>
+        </geometry>
+      </visual>
+      <collision>
+        <origin xyz="0.000000 0.000000 0.000000" rpy="0.000000 0.000000 -0.607892"/>
+        <geometry>
+          <mesh filename="package://6DOF_URDF_description/meshes/6DOF_URDF/Gripper_collision.stl" scale="0.01 0.01 0.01"/>
         </geometry>
       </collision>
@@ -132,34 +147,43 @@
     <joint name="${prefix}Revolute_5" type="revolute">
       <parent link="${prefix}base_link"/>
-      <child link="${prefix}Base_Motor"/>
-      <origin xyz="-0.048850 0.117229 0.068000" rpy="0.000000 0.000000 0.000000"/>
+      <child link="${prefix}Shoulder"/>
+      <origin xyz="0.000000 0.000000 -0.051500" rpy="0.000000 0.000000 0.000000"/>
       <axis xyz="0.000000 0.000000 1.000000"/>
       <limit lower="0.000000" upper="6.283185" effort="100.0" velocity="1.00"/>
     </joint>
     <joint name="${prefix}Revolute_13" type="revolute">
-      <parent link="${prefix}Base_Motor"/>
-      <child link="${prefix}UA_Motor"/>
-      <origin xyz="0.076040 -0.153400 -0.055062" rpy="-1.570796 0.000000 0.000000"/>
-      <axis xyz="0.000000 0.000000 1.000000"/>
-      <limit lower="0.000000" upper="6.283185" effort="100.0" velocity="1.00"/>
-    </joint>
-    <joint name="${prefix}Rigid_25" type="fixed">
-      <parent link="${prefix}UA_Motor"/>
-      <child link="${prefix}Elbow_Connector_Passive"/>
-      <origin xyz="-0.140442 -0.202376 0.018900" rpy="0.000000 0.000000 -0.698132"/>
+      <parent link="${prefix}Shoulder"/>
+      <child link="${prefix}UA"/>
+      <origin xyz="-0.007100 -0.149900 0.111900" rpy="1.570796 0.000000 0.086342"/>
+      <axis xyz="0.000000 0.000000 1.000000"/>
+      <limit lower="0.000000" upper="6.283185" effort="100.0" velocity="1.00"/>
+    </joint>
+    <joint name="${prefix}Revolute_29" type="revolute">
+      <parent link="${prefix}UA"/>
+      <child link="${prefix}Elbow"/>
+      <origin xyz="0.133252 0.154914 -0.036000" rpy="0.000000 0.000000 0.000000"/>
+      <axis xyz="0.000000 0.000000 1.000000"/>
+      <limit lower="0.000000" upper="6.283185" effort="100.0" velocity="1.00"/>
     </joint>
     <joint name="${prefix}Revolute_37" type="revolute">
-      <parent link="${prefix}Elbow_Connector_Passive"/>
-      <child link="${prefix}Roll_Housing"/>
-      <origin xyz="0.106612 0.079606 -0.186510" rpy="-1.570796 0.000000 -0.610865"/>
+      <parent link="${prefix}Elbow"/>
+      <child link="${prefix}Roll"/>
+      <origin xyz="-0.015463 0.083655 -0.071500" rpy="1.570796 -0.214197 -1.161568"/>
       <axis xyz="0.000000 0.000000 1.000000"/>
       <limit lower="0.000000" upper="6.283185" effort="100.0" velocity="1.00"/>
     </joint>
     <joint name="${prefix}Revolute_43" type="revolute">
-      <parent link="${prefix}Roll_Housing"/>
-      <child link="${prefix}20mm"/>
-      <origin xyz="0.251183 -0.314427 0.170791" rpy="1.570796 -1.308997 0.000000"/>
-      <axis xyz="0.000000 0.000000 1.000000"/>
-      <limit lower="0.000000" upper="6.283185" effort="100.0" velocity="1.00"/>
+      <parent link="${prefix}Roll"/>
+      <child link="${prefix}Yaw"/>
+      <origin xyz="0.008683 0.049748 0.186000" rpy="1.570796 1.158599 -0.289463"/>
+      <axis xyz="0.000000 0.000000 1.000000"/>
+      <limit lower="0.000000" upper="6.283185" effort="100.0" velocity="1.00"/>
+    </joint>
+    <joint name="${prefix}Revolute_46" type="continuous">
+      <parent link="${prefix}Yaw"/>
+      <child link="${prefix}Gripper"/>
+      <origin xyz="-0.055454 -0.045134 0.050500" rpy="1.570796 0.110328 -0.887634"/>
+      <axis xyz="0.000000 0.000000 1.000000"/>
+      <limit effort="100.0" velocity="1.00"/>
     </joint>
     <!-- ROS 2 control: generated generic system -->
@@ -179,4 +203,13 @@
         <state_interface name="effort"/>
       </joint>
+      <joint name="${prefix}Revolute_29">
+        <command_interface name="position"/>
+        <command_interface name="velocity"/>
+        <state_interface name="position">
+          <param name="initial_value">0.0</param>
+        </state_interface>
+        <state_interface name="velocity"/>
+        <state_interface name="effort"/>
+      </joint>
       <joint name="${prefix}Revolute_37">
         <command_interface name="position"/>
@@ -189,4 +222,13 @@
       </joint>
       <joint name="${prefix}Revolute_43">
+        <command_interface name="position"/>
+        <command_interface name="velocity"/>
+        <state_interface name="position">
+          <param name="initial_value">0.0</param>
+        </state_interface>
+        <state_interface name="velocity"/>
+        <state_interface name="effort"/>
+      </joint>
+      <joint name="${prefix}Revolute_46">
         <command_interface name="position"/>
         <command_interface name="velocity"/>
